Commit message: Additional models, and laser added to husky

File: pfms-ros/husky/husky_description/urdf/husky_macro.urdf.xacro (robot description, xacro)
@@ -1,5 +1,5 @@
 <?xml version="1.0"?>
 <robot xmlns:xacro="http://ros.org/wiki/xacro">
-  <xacro:arg name="laser_enabled" default="false" />
+  <xacro:arg name="laser_enabled" default="true" />
   <xacro:arg name="laser_xyz" default="$(optenv HUSKY_LMS1XX_XYZ 0.2206 0.0 0.00635)" />
   <xacro:arg name="laser_rpy" default="$(optenv HUSKY_LMS1XX_RPY 0.0 0.0 0.0)" />
@@ -10,4 +10,5 @@
   <xacro:property name="husky_front_bumper_extend" value="$(optenv HUSKY_FRONT_BUMPER_EXTEND 0)" />
   <xacro:property name="husky_rear_bumper_extend" value="$(optenv HUSKY_REAR_BUMPER_EXTEND 0)" />
+  <xacro:arg name="robot_name" default="" />
   <xacro:arg name="robot_namespace" default="/" />
   <xacro:arg name="is_sim" default="false" />
@@ -97,7 +98,7 @@
     </xacro:husky_wheel>
     <xacro:husky_decorate />
-    <!-- <xacro:if value="$(arg laser_enabled)">
-      <xacro:sick_lms1xx_mount prefix="base"/>
-      <xacro:sick_lms1xx frame="base_laser" topic="scan" robot_namespace="$(arg robot_namespace)"/>
+    <xacro:if value="$(arg laser_enabled)">
+      <!-- <xacro:sick_lms1xx_mount prefix="base"/>
+      <xacro:sick_lms1xx frame="base_laser" topic="scan" robot_namespace="$(arg robot_namespace)"/> -->
       <joint name="laser_mount_joint" type="fixed">
         <origin xyz="$(arg laser_xyz)" rpy="$(arg laser_rpy)" />
@@ -105,5 +106,6 @@
         <child link="base_laser_mount" />
       </joint>
-    </xacro:if> -->
+      <link name="base_laser_mount"/>
+    </xacro:if>
     <!--
       top sensor arch; include this if we have realsense enabled
@@ -178,3 +180,39 @@
     </ros2_control>
   </xacro:macro>
+  <gazebo reference="base_laser_mount">
+    <sensor type='ray' name='laser'>
+      <pose>0 0 0 0 0 0</pose>
+      <visualize>false</visualize>
+      <update_rate>30</update_rate>
+      <always_on>true</always_on>
+      <ray>
+        <scan>
+          <horizontal>
+            <samples>640</samples>
+            <resolution>1</resolution>
+            <min_angle>-1.5707</min_angle>
+            <max_angle>1.5707</max_angle>
+          </horizontal>
+        </scan>
+        <range>
+          <min>0.10</min>
+          <max>30.0</max>
+          <resolution>0.01</resolution>
+        </range>
+        <noise>
+          <type>gaussian</type>
+          <mean>0.0</mean>
+          <stddev>0.01</stddev>
+        </noise>
+      </ray>
+      <plugin name="laser_sensor" filename="libgazebo_ros_ray_sensor.so">
+          <ros>
+            <namespace>/$(arg robot_name)</namespace>
+            <remapping>~/out:=laserscan</remapping>
+          </ros>
+          <frame_name>$(arg robot_name)/base_laser_mount</frame_name>
+          <output_type>sensor_msgs/LaserScan</output_type>
+      </plugin>
+    </sensor>
+  </gazebo>
 </robot>

Commit message: files for a3

File: pfms-ros/husky/husky_description/urdf/husky_macro.urdf.xacro (robot description, xacro)
@@ -101,10 +101,10 @@
       <!-- <xacro:sick_lms1xx_mount prefix="base"/>
       <xacro:sick_lms1xx frame="base_laser" topic="scan" robot_namespace="$(arg robot_namespace)"/> -->
-      <joint name="laser_mount_joint" type="fixed">
-        <origin xyz="$(arg laser_xyz)" rpy="$(arg laser_rpy)" />
-        <parent link="top_plate_link" />
-        <child link="base_laser_mount" />
-      </joint>
-      <link name="base_laser_mount"/>
+      <joint name="${prefix}laser_joint" type="fixed">
+        <origin xyz="-${base_x_size/2+0.05} 0 ${base_z_size+0.05}" rpy="$(arg laser_rpy)" />
+        <parent link="${prefix}base_link" />
+        <child link="${prefix}laser_link" />
+      </joint>
+      <link name="${prefix}laser_link"/>
     </xacro:if>
     <!--
@@ -180,8 +180,8 @@
     </ros2_control>
   </xacro:macro>
-  <gazebo reference="base_laser_mount">
+<gazebo reference="laser_link">
     <sensor type='ray' name='laser'>
       <pose>0 0 0 0 0 0</pose>
-      <visualize>false</visualize>
+      <visualize>true</visualize>
       <update_rate>30</update_rate>
       <always_on>true</always_on>
@@ -211,5 +211,5 @@
             <remapping>~/out:=laserscan</remapping>
           </ros>
-          <frame_name>$(arg robot_name)/base_laser_mount</frame_name>
+          <frame_name>$(arg robot_name)laser_link</frame_name>
           <output_type>sensor_msgs/LaserScan</output_type>
       </plugin>

Commit message: working version of the rviz loading

File: pfms-ros/husky/husky_description/urdf/husky_macro.urdf.xacro (robot description, xacro)
@@ -4,4 +4,6 @@
   <xacro:arg name="laser_xyz" default="$(optenv HUSKY_LMS1XX_XYZ 0.2206 0.0 0.00635)" />
   <xacro:arg name="laser_rpy" default="$(optenv HUSKY_LMS1XX_RPY 0.0 0.0 0.0)" />
+  <xacro:arg name="sonar_right_rpy" default="$(optenv HUSKY_SONAR_RIGHT_RPY 0.0 0.0 -1.57079632679)" />
+  <xacro:arg name="sonar_left_rpy" default="$(optenv HUSKY_SONAR_LEFT_RPY 0.0 0.0 1.57079632679)" />
   <xacro:arg name="realsense_enabled" default="false" />
   <xacro:arg name="realsense_xyz" default="$(optenv HUSKY_REALSENSE_XYZ 0 0 0)" />
@@ -107,10 +109,22 @@
       </joint>
       <link name="${prefix}laser_link"/>
-      <joint name="${prefix}sonar_joint" type="fixed">
-        <origin xyz="-${base_x_size/2} 0 ${base_z_size+0.08}" rpy="$(arg laser_rpy)" />
+      <joint name="${prefix}sonar_front_joint" type="fixed">
+        <origin xyz="0 0 ${base_z_size+0.08}" rpy="$(arg laser_rpy)" />
         <parent link="${prefix}base_link" />
-        <child link="${prefix}sonar_link" />
-      </joint>
-      <link name="${prefix}sonar_link"/>
+        <child link="${prefix}sonar_front_link" />
+      </joint>
+      <link name="${prefix}sonar_front_link"/>
+      <joint name="${prefix}sonar_right_joint" type="fixed">
+        <origin xyz="0 0 ${base_z_size+0.08}" rpy="$(arg sonar_right_rpy)" />
+        <parent link="${prefix}base_link" />
+        <child link="${prefix}sonar_right_link" />
+      </joint>
+      <link name="${prefix}sonar_right_link"/>
+      <joint name="${prefix}sonar_left_joint" type="fixed">
+        <origin xyz="0 0 ${base_z_size+0.08}" rpy="$(arg sonar_left_rpy)" />
+        <parent link="${prefix}base_link" />
+        <child link="${prefix}sonar_left_link" />
+      </joint>
+      <link name="${prefix}sonar_left_link"/>
     </xacro:if>
     <!--
@@ -223,6 +237,6 @@
   </gazebo>
   <!-- Sonar sensor -->
-  <gazebo reference="sonar_link">
-    <sensor name="sonar" type="ray">
+  <gazebo reference="sonar_front_link">
+    <sensor name="sonar_front" type="ray">
       <always_on>true</always_on>
       <visualize>true</visualize>
@@ -254,11 +268,94 @@
         </noise>
       </ray>
-      <plugin name="husky_sonar" filename="libgazebo_ros_ray_sensor.so">
+      <plugin name="husky_sonar_front" filename="libgazebo_ros_ray_sensor.so">
         <ros>
-          <remapping>~/out:=$(arg robot_name)/sonar</remapping>
+          <remapping>~/out:=$(arg robot_name)/sonar_front</remapping>
         </ros>
         <output_type>sensor_msgs/Range</output_type>
         <radiation_type>ultrasound</radiation_type>
-        <frame_name>sonar_link</frame_name>
+        <frame_name>sonar_front_link</frame_name>
+      </plugin>
+    </sensor>
+  </gazebo>
+  <!-- Sonar sensor -->
+  <gazebo reference="sonar_right_link">
+    <sensor name="sonar_right" type="ray">
+      <always_on>true</always_on>
+      <visualize>true</visualize>
+      <update_rate>60</update_rate>
+      <ray>
+        <scan>
+          <horizontal>
+            <samples>3</samples>
+            <resolution>1</resolution>
+            <min_angle>-${M_PI * 1.5/180}</min_angle>
+            <max_angle>${M_PI * 1.5/180}</max_angle>
+          </horizontal>
+          <vertical>
+            <samples>3</samples>
+            <resolution>1</resolution>
+            <min_angle>-${M_PI * 1.5/180}</min_angle>
+            <max_angle>${M_PI * 1.5/180}</max_angle>
+          </vertical>
+        </scan>
+        <range>
+          <min>0.02</min>
+          <max>20</max>
+          <resolution>0.01</resolution>
+        </range>
+        <noise>
+          <type>gaussian</type>
+          <mean>0.0</mean>
+          <stddev>0.01</stddev>
+        </noise>
+      </ray>
+      <plugin name="husky_sonar_right" filename="libgazebo_ros_ray_sensor.so">
+        <ros>
+          <remapping>~/out:=$(arg robot_name)/sonar_right</remapping>
+        </ros>
+        <output_type>sensor_msgs/Range</output_type>
+        <radiation_type>ultrasound</radiation_type>
+        <frame_name>sonar_right_link</frame_name>
+      </plugin>
+    </sensor>
+  </gazebo>
+  <gazebo reference="sonar_left_link">
+    <sensor name="sonar_left" type="ray">
+      <always_on>true</always_on>
+      <visualize>true</visualize>
+      <update_rate>60</update_rate>
+      <ray>
+        <scan>
+          <horizontal>
+            <samples>3</samples>
+            <resolution>1</resolution>
+            <min_angle>-${M_PI * 1.5/180}</min_angle>
+            <max_angle>${M_PI * 1.5/180}</max_angle>
+          </horizontal>
+          <vertical>
+            <samples>3</samples>
+            <resolution>1</resolution>
+            <min_angle>-${M_PI * 1.5/180}</min_angle>
+            <max_angle>${M_PI * 1.5/180}</max_angle>
+          </vertical>
+        </scan>
+        <range>
+          <min>0.02</min>
+          <max>20</max>
+          <resolution>0.01</resolution>
+        </range>
+        <noise>
+          <type>gaussian</type>
+          <mean>0.0</mean>
+          <stddev>0.01</stddev>
+        </noise>
+      </ray>
+      <plugin name="husky_sonar_left" filename="libgazebo_ros_ray_sensor.so">
+        <ros>
+          <remapping>~/out:=$(arg robot_name)/sonar_left</remapping>
+        </ros>
+        <output_type>sensor_msgs/Range</output_type>
+        <radiation_type>ultrasound</radiation_type>
+        <frame_name>sonar_left_link</frame_name>
       </plugin>
     </sensor>
