Commit message: drone upgrade

File: pfms-ros/sjtu_drone/sjtu_drone_description/urdf/sjtu_drone.urdf (robot description, URDF)
Before this commit: robot sjtu_drone, 4 links, 3 joints
Links:
- added link base_footprint
Joints:
- added joint base_footprint_joint: type fixed, parent base_footprint, child base_link, origin xyz=0 0 0 rpy=0 0 0
- joint bottom_cam_joint: origin xyz=0 0 0 rpy=0 1.570796326794897 0 -> xyz=0 0 0 rpy=0 1.570796326795 0
- joint sonar_joint: origin xyz=0 0 0 rpy=0 1.570796326794897 0 -> xyz=0 0 0 rpy=0 1.570796326795 0

File: pfms-ros/sjtu_drone/sjtu_drone_description/urdf/sjtu_drone.urdf.xacro (robot description, xacro)
@@ -1,5 +1,18 @@
 <?xml version="1.0" ?>
-<robot name="sjtu_drone"
-  xmlns:xacro="http://ros.org/wiki/xacro">
+<robot name="sjtu_drone" xmlns:xacro="http://www.ros.org/wiki/xacro">
+<!-- https://answers.ros.org/question/379014/passing-outside-parameters-into-urdf-file-using-xacro/ -->
+  <!-- Need argument to get from launch file -->
+  <xacro:arg name="params_path" default="$(find sjtu_drone_bringup)/config/drone.yaml"/>
+  <!-- Need seperate property for xacro inorder processing -->
+  <xacro:property name="params_path" value="$(arg params_path)"/>
+  <!-- Read in the yaml dict as mp (short for model parameters) -->
+  <xacro:property name="mp" value="${xacro.load_yaml(params_path)}"/>
+  <xacro:property name="M_PI" value="3.14159265359" />
+  <link name="base_footprint"/>
+  <joint name="base_footprint_joint" type="fixed">
+    <origin rpy="0 0 0" xyz="0 0 0"/>
+    <parent link="base_footprint"/>
+    <child link="base_link"/>
+  </joint>
   <link name="base_link">
     <inertial>
@@ -26,9 +39,9 @@
     <parent link="base_link" />
     <child link="sonar_link" />
-    <origin rpy="0 1.570796326794897 0" xyz="0 0 0"/>
+    <origin rpy="0 ${M_PI/2} 0" xyz="0 0 0"/>
   </joint>
   <link name="sonar_link"/>
   <joint name="front_cam_joint" type="fixed">
-    <origin rpy="0 0 0" xyz="0.3 0 0"/>
+    <origin rpy="0 0 0" xyz="0.2 0 0"/>
     <parent link="base_link" />
     <child link="front_cam_link" />
@@ -36,5 +49,5 @@
   <link name="front_cam_link"/>
   <joint name="bottom_cam_joint" type="fixed">
-    <origin rpy="0 1.570796326794897 0" xyz="0 0 0"/>
+    <origin rpy="0 ${M_PI/2} 0" xyz="0 0 0"/>
     <parent link="base_link" />
     <child link="bottom_cam_link" />
@@ -50,32 +63,42 @@
   <gazebo>
     <plugin name='simple_drone' filename='libplugin_drone.so'>
+      <ros>
+        <namespace>${mp['namespace']}</namespace>
+        <remapping>cmd_vel:=cmd_vel</remapping>
+        <remapping>imu:=imu</remapping>
+        <remapping>sonar:=sonar</remapping>
+        <remapping>camera_front:=camera_front</remapping>
+        <remapping>camera_bottom:=camera_bottom</remapping>
+        <remapping>camera_front_info:=camera_front_info</remapping>
+        <remapping>camera_bottom_info:=camera_bottom_info</remapping>
+        <remapping>gps:=gps</remapping>
+      </ros>
       <bodyName>base_link</bodyName>
-      <rosNamespace>drone</rosNamespace>
-      <imuTopic>imu</imuTopic>
-      <rollpitchProportionalGain>10.0</rollpitchProportionalGain>
-      <rollpitchDifferentialGain>5.0</rollpitchDifferentialGain>
-      <rollpitchLimit>0.5</rollpitchLimit>
-      <yawProportionalGain>2.0</yawProportionalGain>
-      <yawDifferentialGain>1.0</yawDifferentialGain>
-      <yawLimit>1.5</yawLimit>
-      <velocityXYProportionalGain>5.0</velocityXYProportionalGain>
-      <velocityXYDifferentialGain>2.3</velocityXYDifferentialGain>
-      <velocityXYLimit>2</velocityXYLimit>
-      <velocityZProportionalGain>5.0</velocityZProportionalGain>
-      <velocityZIntegralGain>0.0</velocityZIntegralGain>
-      <velocityZDifferentialGain>1.0</velocityZDifferentialGain>
-      <velocityZLimit>-1</velocityZLimit>
-      <positionXYProportionalGain>1.1</positionXYProportionalGain>
-      <positionXYDifferentialGain>0.0</positionXYDifferentialGain>
-      <positionXYIntegralGain>0.0</positionXYIntegralGain>
-      <positionXYLimit>5</positionXYLimit>
-      <positionZProportionalGain>1.0</positionZProportionalGain>
-      <positionZDifferentialGain>0.2</positionZDifferentialGain>
-      <positionZIntegralGain>0.0</positionZIntegralGain>
-      <positionZLimit>-1</positionZLimit>
-      <maxForce>30</maxForce>
-      <motionSmallNoise>0.05</motionSmallNoise>
-      <motionDriftNoise>0.03</motionDriftNoise>
-      <motionDriftNoiseTime>5.0</motionDriftNoiseTime>
+      <pub_odom>true</pub_odom>
+      <rollpitchProportionalGain>${mp['rollpitchProportionalGain']}</rollpitchProportionalGain>
+      <rollpitchDifferentialGain>${mp['rollpitchDifferentialGain']}</rollpitchDifferentialGain>
+      <rollpitchLimit>${mp['rollpitchLimit']}</rollpitchLimit>
+      <yawProportionalGain>${mp['yawProportionalGain']}</yawProportionalGain>
+      <yawDifferentialGain>${mp['yawDifferentialGain']}</yawDifferentialGain>
+      <yawLimit>${mp['yawLimit']}</yawLimit>
+      <velocityXYProportionalGain>${mp['velocityXYProportionalGain']}</velocityXYProportionalGain>
+      <velocityXYDifferentialGain>${mp['velocityXYDifferentialGain']}</velocityXYDifferentialGain>
+      <velocityXYLimit>${mp['velocityXYLimit']}</velocityXYLimit>
+      <velocityZProportionalGain>${mp['velocityZProportionalGain']}</velocityZProportionalGain>
+      <velocityZIntegralGain>${mp['velocityZIntegralGain']}</velocityZIntegralGain>
+      <velocityZDifferentialGain>${mp['velocityZDifferentialGain']}</velocityZDifferentialGain>
+      <velocityZLimit>${mp['velocityZLimit']}</velocityZLimit>
+      <positionXYProportionalGain>${mp['positionXYProportionalGain']}</positionXYProportionalGain>
+      <positionXYDifferentialGain>${mp['positionXYDifferentialGain']}</positionXYDifferentialGain>
+      <positionXYIntegralGain>${mp['positionXYIntegralGain']}</positionXYIntegralGain>
+      <positionXYLimit>${mp['positionXYLimit']}</positionXYLimit>
+      <positionZProportionalGain>${mp['positionZProportionalGain']}</positionZProportionalGain>
+      <positionZDifferentialGain>${mp['positionZDifferentialGain']}</positionZDifferentialGain>
+      <positionZIntegralGain>${mp['positionZIntegralGain']}</positionZIntegralGain>
+      <positionZLimit>${mp['positionZLimit']}</positionZLimit>
+      <maxForce>${mp['maxForce']}</maxForce>
+      <motionSmallNoise>${mp['motionSmallNoise']}</motionSmallNoise>
+      <motionDriftNoise>${mp['motionDriftNoise']}</motionDriftNoise>
+      <motionDriftNoiseTime>${mp['motionDriftNoiseTime']}</motionDriftNoiseTime>
     </plugin>
   </gazebo>
@@ -88,7 +111,4 @@
       <update_rate> 100 </update_rate>
       <pose> 0 0 0 0 0 0 </pose>
-      <plugin name='imu' filename='libgazebo_ros_imu_sensor.so'>
-        <initial_orientation_as_reference>false</initial_orientation_as_reference>
-      </plugin>
       <imu>
         <noise>
@@ -96,20 +116,28 @@
           <rate>
             <mean> 0 </mean>
-            <stddev> 0 </stddev>
+            <stddev> 0.01 </stddev>
           </rate>
           <accel>
             <mean> 0 </mean>
-            <stddev> 0.00 </stddev>
+            <stddev> 0.01 </stddev>
           </accel>
         </noise>
       </imu>
-    </sensor>
-  </gazebo>
-  <!-- Sonar sensor in 5fps -->
+      <plugin name='imu' filename='libgazebo_ros_imu_sensor.so'>
+        <ros>
+          <namespace>${mp['namespace']}</namespace>
+          <!-- <remapping>imu:=imu</remapping> -->
+        </ros>
+        <initial_orientation_as_reference>false</initial_orientation_as_reference>
+        <frame_name>${mp['namespace']}/base_link</frame_name>
+      </plugin>
+    </sensor>
+  </gazebo>
+  <!-- Sonar sensor in 100fps -->
   <gazebo reference="sonar_link">
     <sensor name="sonar" type="ray">
-      <always_on>true</always_on>
-      <visualize>true</visualize>
-      <update_rate>5</update_rate>
+      <always_on>1</always_on>
+      <visualize>1</visualize>
+      <update_rate>30</update_rate>
       <ray>
         <scan>
@@ -140,9 +168,10 @@
       <plugin name="sonar" filename="libgazebo_ros_ray_sensor.so">
         <ros>
-          <remapping>~/out:=sonar</remapping>
-        </ros>
+          <namespace>${mp['namespace']}</namespace>
+          <!-- <remapping>~/out:=sonar</remapping> -->
+        </ros>
+        <frame_name>${mp['namespace']}/sonar_link</frame_name>
         <output_type>sensor_msgs/Range</output_type>
         <radiation_type>ultrasound</radiation_type>
-        <frame_name>sonar_link</frame_name>
       </plugin>
     </sensor>
@@ -150,4 +179,7 @@
   <gazebo reference="front_cam_link">
     <sensor name="front_camera" type="camera">
+      <always_on>1</always_on>
+      <visualize>1</visualize>
+      <update_rate>60</update_rate>
       <camera>
         <horizontal_fov>2.09</horizontal_fov>
@@ -164,17 +196,15 @@
           <type>gaussian</type>
           <mean>0.0</mean>
-          <stddev>0.005</stddev>
+          <stddev>0.01</stddev>
         </noise>
       </camera>
-      <always_on>1</always_on>
-      <update_rate>60</update_rate>
-      <visualize>true</visualize>
       <plugin name="camera_front" filename="libgazebo_ros_camera.so">
         <ros>
-          <remapping>image_raw:=camera_front</remapping>
-          <remapping>camera_info:=camera_front_info</remapping>
-        </ros>
+          <namespace>${mp['namespace']}</namespace>
+          <!-- <remapping>~/image_raw:=camera_front</remapping>
+          <remapping>~/camera_info:=camera_front_info</remapping> -->
+        </ros>
+        <frame_name>${mp['namespace']}/front_cam_link</frame_name>
         <camera_name>front</camera_name>
-        <frame_name>front_cam_link</frame_name>
         <hack_baseline>0.07</hack_baseline>
       </plugin>
@@ -184,4 +214,7 @@
   <gazebo reference="bottom_cam_link">
     <sensor name="down_camera" type="camera">
+      <always_on>1</always_on>
+      <visualize>1</visualize>
+      <update_rate>15</update_rate>
       <camera>
         <horizontal_fov>1.047</horizontal_fov>
@@ -198,17 +231,15 @@
           <type>gaussian</type>
           <mean>0.0</mean>
-          <stddev>0.005</stddev>
+          <stddev>0.01</stddev>
         </noise>
       </camera>
-      <always_on>1</always_on>
-      <update_rate>15</update_rate>
-      <visualize>true</visualize>
       <plugin name="camera_bottom" filename="libgazebo_ros_camera.so">
         <ros>
-          <remapping>image_raw:=camera_bottom</remapping>
-          <remapping>camera_info:=camera_bottom_info</remapping>
-        </ros>
+          <namespace>${mp['namespace']}</namespace>
+          <!-- <remapping>image_raw:=camera_bottom</remapping>
+          <remapping>camera_info:=camera_bottom_info</remapping> -->
+        </ros>
+        <frame_name>${mp['namespace']}/bottom_cam_link</frame_name>
         <camera_name>bottom</camera_name>
-        <frame_name>bottom_cam_link</frame_name>
         <hack_baseline>0.07</hack_baseline>
       </plugin>
@@ -217,5 +248,5 @@
   <gazebo reference="base_link">
     <sensor name="gps" type="gps">
-      <always_on>true</always_on>
+      <always_on>1</always_on>
       <update_rate>30</update_rate>
       <gps>
@@ -237,7 +268,8 @@
       <plugin name="gps" filename="libgazebo_ros_gps_sensor.so">
         <ros>
-          <namespace>/gps</namespace>
-          <remapping>~/out:=data</remapping>
-        </ros>
+          <namespace>${mp['namespace']}</namespace>
+          <remapping>~/out:=~/nav</remapping>
+        </ros>
+        <frame_name>${mp['namespace']}/base_link</frame_name>
       </plugin>
     </sensor>
@@ -248,5 +280,5 @@
         <visualize>false</visualize>
         <update_rate>30</update_rate>
-        <always_on>true</always_on>
+        <always_on>1</always_on>
         <ray>
           <scan>
@@ -271,11 +303,27 @@
         <plugin name="gazebo_ros_head_hokuyo_controller" filename="libgazebo_ros_ray_sensor.so">
           <ros>
-            <namespace>/sjtu_drone</namespace>
-            <remapping>~/out:=laserscan</remapping>
+	    <namespace>${mp['namespace']}</namespace>
+	    <remapping>~/out:=~/laserscan</remapping>
           </ros>
           <output_type>sensor_msgs/LaserScan</output_type>
-          <frame_name>laser_link</frame_name>
+          <frame_name>${mp['namespace']}/laser_link</frame_name>
         </plugin>
       </sensor>
   </gazebo>
+  <gazebo reference="base_link">
+    <sensor name="collision_sensor" type="contact">
+      <update_rate>100.0</update_rate>
+      <always_on>true</always_on>
+      <contact>
+        <collision>base_footprint_fixed_joint_lump__sjtu_drone_collision_collision</collision>
+      </contact>
+      <plugin name="collision_plugin" filename="libgazebo_ros_bumper.so">
+        <ros>
+          <namespace>${mp['namespace']}</namespace>
+          <!-- <remapping>bumper_states:=bumper_states</remapping> -->
+        </ros>
+        <frame_name>${mp['namespace']}/base_link</frame_name>
+      </plugin>
+    </sensor>
+  </gazebo>
 </robot>

Commit message: ported sjtu_drone updates

File: pfms-ros/sjtu_drone/sjtu_drone_description/urdf/sjtu_drone.urdf (robot description, URDF)
Before this commit: robot sjtu_drone, 5 links, 4 joints
Links:
- added link laser_link
- link base_link: geometry collision mesh filename=file:///home/student/ros2_ws/install/sjtu_drone_description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; visual mesh filename=file:///home/student/ros2_ws/install/sjtu_drone_description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
Joints:
- added joint laser_joint: type fixed, parent base_link, child laser_link, origin xyz=0 0 +0.2 rpy=0 0 0

File: pfms-ros/sjtu_drone/sjtu_drone_description/urdf/sjtu_drone.urdf.xacro (robot description, xacro)
@@ -73,4 +73,5 @@
         <remapping>camera_bottom_info:=camera_bottom_info</remapping>
         <remapping>gps:=gps</remapping>
+        <remapping>laserscan:=laserscan</remapping>
       </ros>
       <bodyName>base_link</bodyName>
@@ -169,5 +170,5 @@
         <ros>
           <namespace>${mp['namespace']}</namespace>
-          <!-- <remapping>~/out:=sonar</remapping> -->
+          <remapping>~/out:=sonar</remapping>
         </ros>
         <frame_name>${mp['namespace']}/sonar_link</frame_name>
@@ -303,6 +304,6 @@
         <plugin name="gazebo_ros_head_hokuyo_controller" filename="libgazebo_ros_ray_sensor.so">
           <ros>
-	    <namespace>${mp['namespace']}</namespace>
-	    <remapping>~/out:=~/laserscan</remapping>
+            <namespace>${mp['namespace']}</namespace>
+            <remapping>~/out:=laserscan</remapping>
           </ros>
           <output_type>sensor_msgs/LaserScan</output_type>
