Commit message: Correction to move audi/quad

File: pfms-ros/sjtu_drone/sjtu_drone_description/urdf/sjtu_drone.urdf.xacro (robot description, xacro)
@@ -30,5 +30,5 @@
   <link name="sonar_link"/>
   <joint name="front_cam_joint" type="fixed">
-    <origin rpy="0 0 0" xyz="0.2 0 0"/>
+    <origin rpy="0 0 0" xyz="0.3 0 0"/>
     <parent link="base_link" />
     <child link="front_cam_link" />
@@ -246,5 +246,5 @@
       <sensor type="ray" name="laser">
         <pose>0 0 0 0 0 0</pose>
-        <visualize>true</visualize>
+        <visualize>false</visualize>
         <update_rate>30</update_rate>
         <always_on>true</always_on>
@@ -252,5 +252,5 @@
           <scan>
             <horizontal>
-              <samples>1800</samples>
+              <samples>360</samples>
               <resolution>1</resolution>
               <min_angle>-3.14167</min_angle>

Commit message: fixed the lins being published, could remove things from gazebo_connect

File: pfms-ros/sjtu_drone/sjtu_drone_description/urdf/sjtu_drone.urdf.xacro (robot description, xacro)
@@ -2,54 +2,12 @@
 <robot name="sjtu_drone"
   xmlns:xacro="http://ros.org/wiki/xacro">
-  <link name="base_link">
-    <inertial>
-      <mass value="1.477"/>
-      <origin rpy="0 0 0" xyz="0 0 0"/>
-      <inertia ixx="0.1152" ixy="0" ixz="0" iyy="0.1152" iyz="0" izz="0.218"/>
-    </inertial>
-    <collision name="sjtu_drone_collision">
-      <origin rpy="0 0 0" xyz="0   0   0.04"/>
-      <geometry>
-        <mesh filename="file://$(find sjtu_drone_description)/models/sjtu_drone/quadrotor_4.stl"/>
-        <!-- <mesh filename="package://sjtu_drone/quadrotor_4.stl"/> -->
-      </geometry>
-    </collision>
-    <visual name="sjtu_drone_visual">
-      <origin rpy="0 0 0" xyz="0   0   0.04"/>
-      <geometry>
-        <mesh filename="file://$(find sjtu_drone_description)/models/sjtu_drone/quadrotor_4.dae"/>
-        <!-- <mesh filename="package://sjtu_drone/quadrotor_4.dae"/> -->
-      </geometry>
-    </visual>
-  </link>
-  <joint name="sonar_joint" type="fixed">
-    <parent link="base_link" />
-    <child link="sonar_link" />
-    <origin rpy="0 1.570796326794897 0" xyz="0 0 0"/>
-  </joint>
-  <link name="sonar_link"/>
-  <joint name="front_cam_joint" type="fixed">
-    <origin rpy="0 0 0" xyz="0.3 0 0"/>
-    <parent link="base_link" />
-    <child link="front_cam_link" />
-  </joint>
-  <link name="front_cam_link"/>
-  <joint name="bottom_cam_joint" type="fixed">
-    <origin rpy="0 1.570796326794897 0" xyz="0 0 0"/>
-    <parent link="base_link" />
-    <child link="bottom_cam_link" />
-  </joint>
-  <link name="bottom_cam_link"/>
-  <!-- Laser -->
-  <joint name="laser_joint" type="fixed">
-    <parent link="base_link" />
-    <child link="laser_link" />
-    <origin xyz="0 0 +0.2" rpy="0 0 0"/>
-  </joint>
-  <link name="laser_link"/>
+  <xacro:arg name="robot_name" default="drone" />
   <gazebo>
     <plugin name='simple_drone' filename='libplugin_drone.so'>
       <bodyName>base_link</bodyName>
-      <rosNamespace>drone</rosNamespace>
+      <robot_name>$(arg robot_name)</robot_name>
+      <ros>
+        <namespace>drone</namespace>
+      </ros>
       <imuTopic>imu</imuTopic>
       <rollpitchProportionalGain>10.0</rollpitchProportionalGain>
@@ -80,4 +38,50 @@
     </plugin>
   </gazebo>
+  <link name="base_link">
+    <inertial>
+      <mass value="1.477"/>
+      <origin rpy="0 0 0" xyz="0 0 0"/>
+      <inertia ixx="0.1152" ixy="0" ixz="0" iyy="0.1152" iyz="0" izz="0.218"/>
+    </inertial>
+    <collision name="sjtu_drone_collision">
+      <origin rpy="0 0 0" xyz="0   0   0.04"/>
+      <geometry>
+        <mesh filename="file://$(find sjtu_drone_description)/models/sjtu_drone/quadrotor_4.stl"/>
+        <!-- <mesh filename="package://sjtu_drone/quadrotor_4.stl"/> -->
+      </geometry>
+    </collision>
+    <visual name="sjtu_drone_visual">
+      <origin rpy="0 0 0" xyz="0   0   0.04"/>
+      <geometry>
+        <mesh filename="file://$(find sjtu_drone_description)/models/sjtu_drone/quadrotor_4.dae"/>
+        <!-- <mesh filename="package://sjtu_drone/quadrotor_4.dae"/> -->
+      </geometry>
+    </visual>
+  </link>
+  <joint name="sonar_joint" type="fixed">
+    <parent link="base_link" />
+    <child link="sonar_link" />
+    <origin rpy="0 1.570796326794897 0" xyz="0 0 0"/>
+  </joint>
+  <link name="sonar_link"/>
+  <joint name="front_cam_joint" type="fixed">
+    <origin rpy="0 0 0" xyz="0.3 0 0"/>
+    <parent link="base_link" />
+    <child link="front_cam_link" />
+  </joint>
+  <link name="front_cam_link"/>
+  <joint name="bottom_cam_joint" type="fixed">
+    <origin rpy="0 1.570796326794897 0" xyz="0 0 0"/>
+    <parent link="base_link" />
+    <child link="bottom_cam_link" />
+  </joint>
+  <link name="bottom_cam_link"/>
+  <!-- Laser -->
+  <joint name="laser_joint" type="fixed">
+    <parent link="base_link" />
+    <child link="laser_link" />
+    <origin xyz="0 0 +0.2" rpy="0 0 0"/>
+  </joint>
+  <link name="laser_link"/>
   <!-- Sensors -->
   <!-- IMU sensor in 100fps -->

Commit message: update for gazebo_fortress

File: pfms-ros/sjtu_drone/sjtu_drone_description/urdf/sjtu_drone.urdf.xacro (robot description, xacro)
@@ -2,4 +2,6 @@
 <robot name="sjtu_drone"
   xmlns:xacro="http://ros.org/wiki/xacro">
+  <!-- namespace property (husky-style gazebo syntax uses a namespace property) -->
+  <xacro:property name="robot_namespace" value="sjtu_drone"/>
   <link name="base_link">
     <inertial>
@@ -51,5 +53,7 @@
     <plugin name='simple_drone' filename='libplugin_drone.so'>
       <bodyName>base_link</bodyName>
-      <rosNamespace>drone</rosNamespace>
+      <ros>
+        <namespace>/${robot_namespace}</namespace>
+      </ros>
       <imuTopic>imu</imuTopic>
       <rollpitchProportionalGain>10.0</rollpitchProportionalGain>
@@ -89,4 +93,7 @@
       <pose> 0 0 0 0 0 0 </pose>
       <plugin name='imu' filename='libgazebo_ros_imu_sensor.so'>
+        <ros>
+          <namespace>/${robot_namespace}</namespace>
+        </ros>
         <initial_orientation_as_reference>false</initial_orientation_as_reference>
       </plugin>
@@ -140,4 +147,5 @@
       <plugin name="sonar" filename="libgazebo_ros_ray_sensor.so">
         <ros>
+          <namespace>/${robot_namespace}</namespace>
           <remapping>~/out:=sonar</remapping>
         </ros>
@@ -172,4 +180,5 @@
       <plugin name="camera_front" filename="libgazebo_ros_camera.so">
         <ros>
+          <namespace>/${robot_namespace}</namespace>
           <remapping>image_raw:=camera_front</remapping>
           <remapping>camera_info:=camera_front_info</remapping>
@@ -206,4 +215,5 @@
       <plugin name="camera_bottom" filename="libgazebo_ros_camera.so">
         <ros>
+          <namespace>/${robot_namespace}</namespace>
           <remapping>image_raw:=camera_bottom</remapping>
           <remapping>camera_info:=camera_bottom_info</remapping>
@@ -237,5 +247,5 @@
       <plugin name="gps" filename="libgazebo_ros_gps_sensor.so">
         <ros>
-          <namespace>/gps</namespace>
+          <namespace>/${robot_namespace}</namespace>
           <remapping>~/out:=data</remapping>
         </ros>
@@ -269,7 +279,7 @@
           </noise>
         </ray>
-        <plugin name="gazebo_ros_head_hokuyo_controller" filename="libgazebo_ros_ray_sensor.so">
+          <plugin name="gazebo_ros_head_hokuyo_controller" filename="libgazebo_ros_ray_sensor.so">
           <ros>
-            <namespace>/sjtu_drone</namespace>
+            <namespace>/${robot_namespace}</namespace>
             <remapping>~/out:=laserscan</remapping>
           </ros>
