Commit message: removed materila warnings

File: pfms-ros/audibot/audibot_description/urdf/audibot.urdf.xacro (robot description, xacro)
@@ -135,5 +135,5 @@
              <box size="0.1 0.1 0.1"/>
           </geometry>
-          <material name="blue"/>
+          <!--material name="blue"/-->
         </visual>
       <inertial>
@@ -154,5 +154,5 @@
              <box size="0.1 0.1 0.1"/>
           </geometry>
-          <material name="blue"/>
+          <!--material name="blue"/-->
         </visual>
       <inertial>
@@ -252,4 +252,5 @@
           <frameName>orange/front_sonar_link</frameName>
           <fov>0.2</fov>
+          <radiation>ultrasound</radiation>
         </plugin>
         <always_on>false</always_on>

Commit message: Updates for ROS2 humble

File: pfms-ros/audibot/audibot_description/urdf/audibot.urdf.xacro (robot description, xacro)
@@ -13,17 +13,27 @@
   <xacro:arg name="pub_tf" default="true" />
   <xacro:arg name="robot_name" default="" />
+  <xacro:arg name="blue" default="false" />
   <gazebo>
     <!-- Simulated vehicle interface -->
     <plugin name="audibot_interface_plugin" filename="libaudibot_interface_plugin.so" >
-      <robotName>$(arg robot_name)</robotName>
-      <pubTf>$(arg pub_tf)</pubTf>
-      <tfFreq>100.0</tfFreq>
+      <robot_name>$(arg robot_name)</robot_name>
+      <pub_tf>$(arg pub_tf)</pub_tf>
+      <tf_freq>100.0</tf_freq>
+      <ros>
+        <namespace>$(arg robot_name)</namespace>
+      </ros>
     </plugin>
     <!-- Publish current joint angles -->
     <plugin name="joint_state_publisher" filename="libgazebo_ros_joint_state_publisher.so">
-        <jointName>
-            steer_fl_joint, steer_fr_joint, wheel_fl_joint, wheel_fr_joint, wheel_rl_joint, wheel_rr_joint
-        </jointName>
-        <updateRate>100</updateRate>
+        <joint_name>steer_fl_joint</joint_name>
+        <joint_name>steer_fr_joint</joint_name>
+        <joint_name>wheel_fl_joint</joint_name>
+        <joint_name>wheel_fr_joint</joint_name>
+        <joint_name>wheel_rl_joint</joint_name>
+        <joint_name>wheel_rr_joint</joint_name>
+        <update_rate>100</update_rate>
+        <ros>
+          <namespace>$(arg robot_name)</namespace>
+        </ros>
     </plugin>
   </gazebo>
@@ -33,5 +43,5 @@
         <origin xyz="0 0 0" rpy="1.57079632679 ${flip * 3.1415926535} 0" />
         <geometry>
-          <mesh filename="package://audibot_description/meshes/wheel.dae" scale="1 1 1" />
+          <mesh filename="file://$(find audibot_description)/meshes/wheel.dae" scale="1 1 1" />
         </geometry>
       </visual>
@@ -60,5 +70,5 @@
         <origin xyz="0 0 0" rpy="1.57079632679 ${flip * pi} 0" />
         <geometry>
-          <mesh filename="package://audibot_description/meshes/wheel.dae" scale="1 1 1" />
+          <mesh filename="file://$(find audibot_description)/meshes/wheel.dae" scale="1 1 1" />
         </geometry>
       </visual>
@@ -103,8 +113,8 @@
       <geometry>
         <xacro:if value="$(arg blue)" >
-          <mesh filename="package://audibot_description/meshes/blue_body.dae" scale="1 1 1" />
+          <mesh filename="file://$(find audibot_description)/meshes/blue_body.dae" scale="1 1 1" />
         </xacro:if>
         <xacro:unless value="$(arg blue)" >
-          <mesh filename="package://audibot_description/meshes/orange_body.dae" scale="1 1 1" />
+          <mesh filename="file://$(find audibot_description)/meshes/orange_body.dae" scale="1 1 1" />
         </xacro:unless>
       </geometry>
@@ -113,5 +123,5 @@
       <origin xyz="0.035 0 0.025" rpy="0 0 0" />
       <geometry>
-        <mesh filename="package://audibot_description/meshes/body_collision.stl" scale="1 1 1" />
+        <mesh filename="file://$(find audibot_description)/meshes/body_collision.stl" scale="1 1 1" />
       </geometry>
     </collision>
@@ -127,43 +137,31 @@
     <child link="base_link"/>
   </joint>
-    <!-- Sensor links and fixed joints -->
-    <link name="front_laser_link">
-        <visual>
-          <origin xyz="0 0 0" rpy="0 0 0"/>
-          <geometry>
-            <!--mesh filename="package://rrbot_description/meshes/hokuyo.dae"/-->
-             <box size="0.1 0.1 0.1"/>
-          </geometry>
-          <!--material name="blue"/-->
-        </visual>
-      <inertial>
-        <mass value="1"/>
-        <inertia ixx="0.001" ixy="0.0" ixz="0.0" iyy="0.001" iyz="0.0" izz="0.001"/>
-      </inertial>
-    </link>
-    <joint name="front_laser_joint" type="fixed">
-      <parent link="base_link"/>
-      <child link="front_laser_link"/>
-      <origin xyz="${body_depth -1.05} 0 0.2" rpy="0 0 0"/>
-    </joint>
-    <link name="front_sonar_link">
-        <visual>
-          <origin xyz="0 0 0" rpy="0 0 0"/>
-          <geometry>
-            <!--mesh filename="package://rrbot_description/meshes/hokuyo.dae"/-->
-             <box size="0.1 0.1 0.1"/>
-          </geometry>
-          <!--material name="blue"/-->
-        </visual>
-      <inertial>
-        <mass value="1"/>
-        <inertia ixx="0.001" ixy="0.0" ixz="0.0" iyy="0.001" iyz="0.0" izz="0.001"/>
-      </inertial>
-    </link>
-    <joint name="front_sonar_joint" type="fixed">
-      <parent link="base_link"/>
-      <child link="front_sonar_link"/>
-      <origin xyz="${body_depth -1.05} 0 0.5" rpy="0 0 0"/>
-    </joint>
+  <!-- Sensor links and fixed joints -->
+  <!--link name="front_laser_link">
+      <visual>
+        <origin xyz="0 0 0" rpy="0 0 0"/>
+        <geometry-->
+          <!--mesh filename="package://rrbot_description/meshes/hokuyo.dae"/-->
+            <!--box size="0.1 0.1 0.1"/>
+        </geometry-->
+        <!--material name="blue"/-->
+      <!--/visual>
+    <inertial>
+      <mass value="1"/>
+      <inertia ixx="0.001" ixy="0.0" ixz="0.0" iyy="0.001" iyz="0.0" izz="0.001"/>
+    </inertial>
+  </link>
+  <joint name="front_laser_joint" type="fixed">
+    <parent link="base_link"/>
+    <child link="front_laser_link"/>
+    <origin xyz="${body_depth -1.05} 0 0.2" rpy="0 0 0"/>
+  </joint-->
+  <!-- Laser -->
+  <joint name="laser_joint" type="fixed">
+    <parent link="base_link" />
+    <child link="laser_link" />
+    <origin xyz="${body_depth -1.05} 0 0.1" rpy="0 0 0"/>
+  </joint>
+  <link name="laser_link"/>
   <xacro:rear_wheel name="rl" x="${-half_wheelbase}" y="${half_rear_track_width}" z="0" flip="1" />
   <xacro:rear_wheel name="rr" x="${-half_wheelbase}" y="${-half_rear_track_width}" z="0" flip="0" />
@@ -191,100 +189,39 @@
     <mu2>${wheel_friction}</mu2>
   </gazebo>
-    <gazebo reference="front_laser_link">
-      <sensor name='front_laser_sensor' type='ray'>
-        <pose>0 0 0 0 0 0</pose>
-        <visualize>false</visualize>
-        <update_rate>30</update_rate>
-        <ray>
-          <scan>
-            <horizontal>
-              <samples>640</samples>
-              <resolution>1</resolution>
-              <min_angle>-1.5707</min_angle>
-              <max_angle>1.5707</max_angle>
-            </horizontal>
-          </scan>
-          <range>
-            <min>0.10</min>
-            <max>30.0</max>
-            <resolution>0.01</resolution>
-          </range>
-          <noise>
-            <type>gaussian</type>
-            <!-- Noise parameters based on published spec for Hokuyo laser
-                 achieving "+-30mm" accuracy at range < 10m.  A mean of 0.0m and
-                 stddev of 0.01m will put 99.7% of samples within 0.03m of the true
-                 reading. -->
-            <mean>0.0</mean>
-            <stddev>0.01</stddev>
-          </noise>
-        </ray>
-        <plugin name="gazebo_ros_head_hokuyo_controller" filename="libgazebo_ros_laser.so">
-            <topicName>/$(arg robot_name)/laser/scan</topicName>
-            <frameName>/$(arg robot_name)/front_laser_link</frameName>
-        </plugin>
-      </sensor>
-    </gazebo>
-    <gazebo reference="front_sonar_link">
-      <sensor name='front_sonar_sensor' type='ray'>
-        <ray>
-          <scan>
-            <horizontal>
-              <samples>1</samples>
-              <resolution>1</resolution>
-              <min_angle>0</min_angle>
-              <max_angle>0</max_angle>
-            </horizontal>
-            <vertical>
-              <samples>1</samples>
-              <min_angle>0</min_angle>
-              <max_angle>0</max_angle>
-            </vertical>
-          </scan>
-          <range>
-            <min>0.2</min>
-            <max>5</max>
-            <resolution>0.2</resolution>
-          </range>
-        </ray>
-        <plugin name='front_sonar_sensor' filename='libgazebo_ros_range.so'>
-          <topicName>/$(arg robot_name)/sonar/range</topicName>
-          <frameName>/$(arg robot_name)/front_sonar_link</frameName>
-          <fov>0.2</fov>
-          <radiation>ultrasound</radiation>
-        </plugin>
-        <always_on>false</always_on>
-        <update_rate>5</update_rate>
-        <visualize>true</visualize>
-      </sensor>
-    </gazebo>
-    <gazebo reference="front_sonar_link">
-      <!-- front camera -->
-      <sensor name="front_camera" type="camera">
-        <camera>
-          <horizontal_fov>2.1</horizontal_fov>
-          <image>
-            <width>640</width>
-            <height>480</height>
-            <format>R8G8B8</format>
-          </image>
-          <clip>
-            <near>0.1</near>
-            <far>100</far>
-          </clip>
-          <noise>
-            <type>gaussian</type>
-            <mean>0.0</mean>
-            <stddev>0.005</stddev>
-          </noise>
-        </camera>
-        <pose> 0.0 0.0 0.1 0 0 0 </pose>
-        <always_on>1</always_on>
-        <update_rate>30</update_rate>
-        <visualize>true</visualize>
-        <plugin name='front_camera' filename='libplugin_ros_cam.so'>
-          <imageTopicName>/$(arg robot_name)/front_camera/image_raw</imageTopicName>
-        </plugin>
-      </sensor>
-    </gazebo>
+  <gazebo reference="laser_link">
+    <sensor type='ray' name='laser'>
+      <pose>0 0 0 0 0 0</pose>
+      <visualize>false</visualize>
+      <update_rate>30</update_rate>
+      <always_on>true</always_on>
+      <ray>
+        <scan>
+          <horizontal>
+            <samples>640</samples>
+            <resolution>1</resolution>
+            <min_angle>-1.5707</min_angle>
+            <max_angle>1.5707</max_angle>
+          </horizontal>
+        </scan>
+        <range>
+          <min>0.10</min>
+          <max>30.0</max>
+          <resolution>0.01</resolution>
+        </range>
+        <noise>
+          <type>gaussian</type>
+          <mean>0.0</mean>
+          <stddev>0.01</stddev>
+        </noise>
+      </ray>
+      <plugin name="laser_sensor" filename="libgazebo_ros_ray_sensor.so">
+          <ros>
+            <namespace>/$(arg robot_name)</namespace>
+            <remapping>~/out:=laserscan</remapping>
+          </ros>
+          <frame_name>$(arg robot_name)/laser_link</frame_name>
+          <output_type>sensor_msgs/LaserScan</output_type>
+      </plugin>
+    </sensor>
+  </gazebo>
 </robot>

Commit message: Added camera to audibot

File: pfms-ros/audibot/audibot_description/urdf/audibot.urdf.xacro (robot description, xacro)
@@ -164,4 +164,10 @@
   </joint>
   <link name="laser_link"/>
+  <joint name="camera_joint" type="fixed">
+    <parent link="base_link" />
+    <child link="camera_link" />
+    <origin xyz="${body_depth -1.05} 0 0.2" rpy="0 0 0"/>
+  </joint>
+  <link name="camera_link"/>
   <xacro:rear_wheel name="rl" x="${-half_wheelbase}" y="${half_rear_track_width}" z="0" flip="1" />
   <xacro:rear_wheel name="rr" x="${-half_wheelbase}" y="${-half_rear_track_width}" z="0" flip="0" />
@@ -225,3 +231,40 @@
     </sensor>
   </gazebo>
+    <gazebo reference="camera_link">
+      <!-- front camera -->
+      <sensor type="camera" name="front_camera">
+        <camera>
+          <horizontal_fov>2.1</horizontal_fov>
+          <image>
+            <width>640</width>
+            <height>480</height>
+            <format>R8G8B8</format>
+          </image>
+          <clip>
+            <near>0.1</near>
+            <far>100</far>
+          </clip>
+          <noise>
+            <type>gaussian</type>
+            <mean>0.0</mean>
+            <stddev>0.005</stddev>
+          </noise>
+        </camera>
+        <visualize>true</visualize>
+        <plugin name='front_camera' filename='libgazebo_ros_camera.so'>
+          <alwaysOn>true</alwaysOn>
+          <updateRate>15.0</updateRate>
+          <cameraName>audibot/camera</cameraName>
+          <imageTopicName>$(arg robot_name)/camera/image_raw</imageTopicName>
+          <cameraInfoTopicName>$(arg robot_name)/camera/camera_info</cameraInfoTopicName>
+          <frameName>camera_link</frameName>
+          <hackBaseline>0.07</hackBaseline>
+          <distortionK1>0.0</distortionK1>
+          <distortionK2>0.0</distortionK2>
+          <distortionK3>0.0</distortionK3>
+          <distortionT1>0.0</distortionT1>
+          <distortionT2>0.0</distortionT2>
+        </plugin>
+      </sensor>
+    </gazebo>
 </robot>

Commit message: changes for a1

File: pfms-ros/audibot/audibot_description/urdf/audibot.urdf.xacro (robot description, xacro)
@@ -14,4 +14,5 @@
   <xacro:arg name="robot_name" default="" />
   <xacro:arg name="blue" default="false" />
+  <xacro:property name="M_PI" value="3.1415926535897931" />
   <gazebo>
     <!-- Simulated vehicle interface -->
@@ -170,4 +171,10 @@
   </joint>
   <link name="camera_link"/>
+  <joint name="sonar_joint" type="fixed">
+    <parent link="base_link" />
+    <child link="sonar_link" />
+    <origin xyz="${body_depth -1.05} 0 0.2" rpy="0 0 0"/>
+  </joint>
+  <link name="sonar_link"/>
   <xacro:rear_wheel name="rl" x="${-half_wheelbase}" y="${half_rear_track_width}" z="0" flip="1" />
   <xacro:rear_wheel name="rr" x="${-half_wheelbase}" y="${-half_rear_track_width}" z="0" flip="0" />
@@ -231,46 +238,88 @@
     </sensor>
   </gazebo>
-    <gazebo reference="camera_link">
-      <!-- front camera -->
-      <sensor type="camera" name="front_camera">
-        <camera>
-          <horizontal_fov>2.1</horizontal_fov>
-          <image>
-            <width>640</width>
-            <height>480</height>
-            <format>R8G8B8</format>
-          </image>
-          <clip>
-            <near>0.1</near>
-            <far>100</far>
-          </clip>
-          <noise>
-            <type>gaussian</type>
-            <mean>0.0</mean>
-            <stddev>0.005</stddev>
-          </noise>
-        </camera>
-        <visualize>true</visualize>
-        <plugin name='front_camera' filename='libgazebo_ros_camera.so'>
-          <ros>
-            <namespace>/$(arg robot_name)</namespace>
-            <!--remapping>~/out:=laserscan</remapping-->
-          </ros>
-          <frame_name>$(arg robot_name)/camera_link</frame_name>
-          <!--output_type>sensor_msgs/LaserScan</output_type-->
-          <alwaysOn>true</alwaysOn>
-          <updateRate>15.0</updateRate>
-          <cameraName>$(arg robot_name)/camera</cameraName>
-          <imageTopicName>$(arg robot_name)/camera/image_raw</imageTopicName>
-          <cameraInfoTopicName>$(arg robot_name)/camera/camera_info</cameraInfoTopicName>
-          <!--frameName>camera_link</frameName-->
-          <hackBaseline>0.07</hackBaseline>
-          <distortionK1>0.0</distortionK1>
-          <distortionK2>0.0</distortionK2>
-          <distortionK3>0.0</distortionK3>
-          <distortionT1>0.0</distortionT1>
-          <distortionT2>0.0</distortionT2>
-        </plugin>
-      </sensor>
-    </gazebo>
+  <gazebo reference="camera_link">
+    <!-- front camera -->
+    <sensor type="camera" name="front_camera">
+      <camera>
+        <horizontal_fov>2.1</horizontal_fov>
+        <image>
+          <width>640</width>
+          <height>480</height>
+          <format>R8G8B8</format>
+        </image>
+        <clip>
+          <near>0.1</near>
+          <far>100</far>
+        </clip>
+        <noise>
+          <type>gaussian</type>
+          <mean>0.0</mean>
+          <stddev>0.005</stddev>
+        </noise>
+      </camera>
+      <visualize>true</visualize>
+      <plugin name='front_camera' filename='libgazebo_ros_camera.so'>
+        <ros>
+          <namespace>/$(arg robot_name)</namespace>
+          <!--remapping>~/out:=laserscan</remapping-->
+        </ros>
+        <frame_name>$(arg robot_name)/camera_link</frame_name>
+        <!--output_type>sensor_msgs/LaserScan</output_type-->
+        <alwaysOn>true</alwaysOn>
+        <updateRate>10.0</updateRate>
+        <cameraName>$(arg robot_name)/camera</cameraName>
+        <imageTopicName>$(arg robot_name)/camera/image_raw</imageTopicName>
+        <cameraInfoTopicName>$(arg robot_name)/camera/camera_info</cameraInfoTopicName>
+        <!--frameName>camera_link</frameName-->
+        <hackBaseline>0.07</hackBaseline>
+        <distortionK1>0.0</distortionK1>
+        <distortionK2>0.0</distortionK2>
+        <distortionK3>0.0</distortionK3>
+        <distortionT1>0.0</distortionT1>
+        <distortionT2>0.0</distortionT2>
+      </plugin>
+    </sensor>
+  </gazebo>
+  <!-- Sonar sensor -->
+  <gazebo reference="sonar_link">
+    <sensor name="sonar" type="ray">
+      <always_on>true</always_on>
+      <visualize>true</visualize>
+      <update_rate>60</update_rate>
+      <ray>
+        <scan>
+          <horizontal>
+            <samples>3</samples>
+            <resolution>1</resolution>
+            <min_angle>-${M_PI * 1.5/180}</min_angle>
+            <max_angle>${M_PI * 1.5/180}</max_angle>
+          </horizontal>
+          <vertical>
+            <samples>3</samples>
+            <resolution>1</resolution>
+            <min_angle>-${M_PI * 1.5/180}</min_angle>
+            <max_angle>${M_PI * 1.5/180}</max_angle>
+          </vertical>
+        </scan>
+        <range>
+          <min>0.02</min>
+          <max>20</max>
+          <resolution>0.01</resolution>
+        </range>
+        <noise>
+          <type>gaussian</type>
+          <mean>0.0</mean>
+          <stddev>0.01</stddev>
+        </noise>
+      </ray>
+      <plugin name="audi_sonar" filename="libgazebo_ros_ray_sensor.so">
+        <ros>
+          <remapping>~/out:=$(arg robot_name)/sonar</remapping>
+        </ros>
+        <output_type>sensor_msgs/Range</output_type>
+        <radiation_type>ultrasound</radiation_type>
+        <frame_name>sonar_link</frame_name>
+      </plugin>
+    </sensor>
+  </gazebo>
 </robot>

File: pfms-ros/husky/husky_description/urdf/husky_macro.urdf.xacro (robot description, xacro)
@@ -10,5 +10,5 @@
   <xacro:property name="husky_front_bumper_extend" value="$(optenv HUSKY_FRONT_BUMPER_EXTEND 0)" />
   <xacro:property name="husky_rear_bumper_extend" value="$(optenv HUSKY_REAR_BUMPER_EXTEND 0)" />
-  <xacro:arg name="robot_name" default="" />
+  <xacro:arg name="robot_name" default="husky" />
   <xacro:arg name="robot_namespace" default="/" />
   <xacro:arg name="is_sim" default="false" />
@@ -102,9 +102,15 @@
       <xacro:sick_lms1xx frame="base_laser" topic="scan" robot_namespace="$(arg robot_namespace)"/> -->
       <joint name="${prefix}laser_joint" type="fixed">
-        <origin xyz="-${base_x_size/2+0.05} 0 ${base_z_size+0.05}" rpy="$(arg laser_rpy)" />
+        <origin xyz="-${base_x_size/2} 0 ${base_z_size+0.05}" rpy="$(arg laser_rpy)" />
         <parent link="${prefix}base_link" />
         <child link="${prefix}laser_link" />
       </joint>
       <link name="${prefix}laser_link"/>
+      <joint name="${prefix}sonar_joint" type="fixed">
+        <origin xyz="-${base_x_size/2} 0 ${base_z_size+0.08}" rpy="$(arg laser_rpy)" />
+        <parent link="${prefix}base_link" />
+        <child link="${prefix}sonar_link" />
+      </joint>
+      <link name="${prefix}sonar_link"/>
     </xacro:if>
     <!--
@@ -211,8 +217,50 @@
             <remapping>~/out:=laserscan</remapping>
           </ros>
-          <frame_name>$(arg robot_name)laser_link</frame_name>
+          <frame_name>laser_link</frame_name>
           <output_type>sensor_msgs/LaserScan</output_type>
       </plugin>
     </sensor>
   </gazebo>
+  <!-- Sonar sensor -->
+  <gazebo reference="sonar_link">
+    <sensor name="sonar" type="ray">
+      <always_on>true</always_on>
+      <visualize>true</visualize>
+      <update_rate>60</update_rate>
+      <ray>
+        <scan>
+          <horizontal>
+            <samples>3</samples>
+            <resolution>1</resolution>
+            <min_angle>-${M_PI * 1.5/180}</min_angle>
+            <max_angle>${M_PI * 1.5/180}</max_angle>
+          </horizontal>
+          <vertical>
+            <samples>3</samples>
+            <resolution>1</resolution>
+            <min_angle>-${M_PI * 1.5/180}</min_angle>
+            <max_angle>${M_PI * 1.5/180}</max_angle>
+          </vertical>
+        </scan>
+        <range>
+          <min>0.02</min>
+          <max>20</max>
+          <resolution>0.01</resolution>
+        </range>
+        <noise>
+          <type>gaussian</type>
+          <mean>0.0</mean>
+          <stddev>0.01</stddev>
+        </noise>
+      </ray>
+      <plugin name="husky_sonar" filename="libgazebo_ros_ray_sensor.so">
+        <ros>
+          <remapping>~/out:=$(arg robot_name)/sonar</remapping>
+        </ros>
+        <output_type>sensor_msgs/Range</output_type>
+        <radiation_type>ultrasound</radiation_type>
+        <frame_name>sonar_link</frame_name>
+      </plugin>
+    </sensor>
+  </gazebo>
 </robot>

File: pfms-ros/sjtu_drone/sjtu_drone_description/urdf/sjtu_drone.urdf.xacro (robot description, xacro)
@@ -45,5 +45,5 @@
     <parent link="base_link" />
     <child link="laser_link" />
-    <origin xyz="0 0 +0.1" rpy="0 0 0"/>
+    <origin xyz="0 0 +0.2" rpy="0 0 0"/>
   </joint>
   <link name="laser_link"/>
@@ -106,5 +106,5 @@
     </sensor>
   </gazebo>
-  <!-- Sonar sensor in 100fps -->
+  <!-- Sonar sensor in 5fps -->
   <gazebo reference="sonar_link">
     <sensor name="sonar" type="ray">
