Commit message: Attempted to fix issues, no solutions

File: pfms-ros/audibot/audibot_description/urdf/audibot.urdf.xacro (robot description, xacro)
@@ -33,5 +33,5 @@
         <joint_name>wheel_rl_joint</joint_name>
         <joint_name>wheel_rr_joint</joint_name>
-        <update_rate>100</update_rate>
+        <update_rate>100</update_rate> s
         <ros>
           <namespace>$(arg robot_name)</namespace>
@@ -313,5 +313,5 @@
         </noise>
       </ray>
-      <plugin name="audi_sonar" filename="libgazebo_ros_ray_sensor.so">
+      <plugin name="sonar" filename="libgazebo_ros_ray_sensor.so">
         <ros>
           <namespace>/$(arg robot_name)</namespace>

File: pfms-ros/husky/husky_description/urdf/husky_macro.urdf.xacro (robot description, xacro)
@@ -6,4 +6,5 @@
   <xacro:arg name="sonar_right_rpy" default="$(optenv HUSKY_SONAR_RIGHT_RPY 0.0 0.0 -1.57079632679)" />
   <xacro:arg name="sonar_left_rpy" default="$(optenv HUSKY_SONAR_LEFT_RPY 0.0 0.0 1.57079632679)" />
+  <xacro:arg name="sonar_back_rpy" default="$(optenv HUSKY_SONAR_LEFT_RPY 0.0 0.0 3.14159)" />
   <xacro:arg name="realsense_enabled" default="false" />
   <xacro:arg name="realsense_xyz" default="$(optenv HUSKY_REALSENSE_XYZ 0 0 0)" />
@@ -127,4 +128,10 @@
       </joint>
       <link name="${prefix}sonar_left_link"/>
+      <joint name="${prefix}sonar_back_joint" type="fixed">
+        <origin xyz="0 0 ${base_z_size+0.08}" rpy="$(arg sonar_back_rpy)" />
+        <parent link="${prefix}base_link" />
+        <child link="${prefix}sonar_back_link" />
+      </joint>
+      <link name="${prefix}sonar_back_link"/>
     </xacro:if>
     <!--
@@ -203,6 +210,6 @@
     <sensor type='ray' name='laser'>
       <pose>0 0 0 0 0 0</pose>
-      <visualize>true</visualize>
-      <update_rate>30</update_rate>
+      <visualize>false</visualize>
+      <update_rate>20</update_rate>
       <always_on>true</always_on>
       <ray>
@@ -361,3 +368,44 @@
     </sensor>
   </gazebo>
+  <gazebo reference="sonar_back_link">
+    <sensor name="sonar_back" type="ray">
+      <always_on>true</always_on>
+      <visualize>true</visualize>
+      <update_rate>60</update_rate>
+      <ray>
+        <scan>
+          <horizontal>
+            <samples>3</samples>
+            <resolution>1</resolution>
+            <min_angle>-${M_PI * 1.5/180}</min_angle>
+            <max_angle>${M_PI * 1.5/180}</max_angle>
+          </horizontal>
+          <vertical>
+            <samples>3</samples>
+            <resolution>1</resolution>
+            <min_angle>-${M_PI * 1.5/180}</min_angle>
+            <max_angle>${M_PI * 1.5/180}</max_angle>
+          </vertical>
+        </scan>
+        <range>
+          <min>0.02</min>
+          <max>20</max>
+          <resolution>0.01</resolution>
+        </range>
+        <noise>
+          <type>gaussian</type>
+          <mean>0.0</mean>
+          <stddev>0.01</stddev>
+        </noise>
+      </ray>
+      <plugin name="husky_sonar_back" filename="libgazebo_ros_ray_sensor.so">
+        <ros>
+          <remapping>~/out:=$(arg robot_name)/sonar_back</remapping>
+        </ros>
+        <output_type>sensor_msgs/Range</output_type>
+        <radiation_type>ultrasound</radiation_type>
+        <frame_name>sonar_back_link</frame_name>
+      </plugin>
+    </sensor>
+  </gazebo>
 </robot>

File: pfms-ros/sjtu_drone/sjtu_drone_description/urdf/sjtu_drone.urdf.xacro (robot description, xacro)
@@ -3,4 +3,5 @@
   xmlns:xacro="http://ros.org/wiki/xacro">
   <xacro:arg name="robot_name" default="drone" />
+  <xacro:property name="M_PI" value="3.14159"/>
   <gazebo>
     <plugin name='simple_drone' filename='libplugin_drone.so'>
@@ -59,10 +60,34 @@
     </visual>
   </link>
-  <joint name="sonar_joint" type="fixed">
-    <parent link="base_link" />
-    <child link="sonar_link" />
+  <joint name="sonar_bottom_joint" type="fixed">
+    <parent link="base_link" />
+    <child link="sonar_bottom_link" />
     <origin rpy="0 1.570796326794897 0" xyz="0 0 0"/>
   </joint>
-  <link name="sonar_link"/>
+  <link name="sonar_bottom_link"/>
+  <joint name="sonar_front_joint" type="fixed">
+    <parent link="base_link" />
+    <child link="sonar_front_link" />
+    <origin rpy="0 0 0" xyz="0 0 0.15"/>
+  </joint>
+  <link name="sonar_front_link"/>
+  <joint name="sonar_right_joint" type="fixed">
+    <parent link="base_link" />
+    <child link="sonar_right_link" />
+    <origin rpy="0 0 -1.57079632679" xyz="0 0 0.15"/>
+  </joint>
+  <link name="sonar_right_link"/>
+  <joint name="sonar_left_joint" type="fixed">
+    <parent link="base_link" />
+    <child link="sonar_left_link" />
+    <origin rpy="0 0 1.57079632679" xyz="0 0 0.15"/>
+  </joint>
+  <link name="sonar_left_link"/>
+  <joint name="sonar_back_joint" type="fixed">
+    <parent link="base_link" />
+    <child link="sonar_back_link" />
+    <origin rpy="0 0 3.14159" xyz="0 0 0.15"/>
+  </joint>
+  <link name="sonar_back_link"/>
   <joint name="front_cam_joint" type="fixed">
     <origin rpy="0 0 0" xyz="0.3 0 0"/>
@@ -112,6 +137,6 @@
   </gazebo>
   <!-- Sonar sensor in 5fps -->
-  <gazebo reference="sonar_link">
-    <sensor name="sonar" type="ray">
+  <gazebo reference="sonar_bottom_link">
+    <sensor name="sonar_bottom" type="ray">
       <always_on>true</always_on>
       <visualize>true</visualize>
@@ -146,9 +171,175 @@
         <ros>
           <namespace>$(arg robot_name)</namespace>
-          <remapping>~/out:=sonar</remapping>
+          <remapping>~/out:=sonar_bottom</remapping>
         </ros>
         <output_type>sensor_msgs/Range</output_type>
         <radiation_type>ultrasound</radiation_type>
-        <frame_name>sonar_link</frame_name>
+        <frame_name>sonar_bottom_link</frame_name>
+      </plugin>
+    </sensor>
+  </gazebo>
+  <!-- Sonar sensor -->
+  <gazebo reference="sonar_front_link">
+    <sensor name="sonar_front" type="ray">
+      <always_on>true</always_on>
+      <visualize>true</visualize>
+      <update_rate>60</update_rate>
+      <ray>
+        <scan>
+          <horizontal>
+            <samples>3</samples>
+            <resolution>1</resolution>
+            <min_angle>-${M_PI * 1.5/180}</min_angle>
+            <max_angle>${M_PI * 1.5/180}</max_angle>
+          </horizontal>
+          <vertical>
+            <samples>3</samples>
+            <resolution>1</resolution>
+            <min_angle>-${M_PI * 1.5/180}</min_angle>
+            <max_angle>${M_PI * 1.5/180}</max_angle>
+          </vertical>
+        </scan>
+        <range>
+          <min>0.02</min>
+          <max>20</max>
+          <resolution>0.01</resolution>
+        </range>
+        <noise>
+          <type>gaussian</type>
+          <mean>0.0</mean>
+          <stddev>0.01</stddev>
+        </noise>
+      </ray>
+      <plugin name="drone_sonar_front" filename="libgazebo_ros_ray_sensor.so">
+        <ros>
+          <remapping>~/out:=$(arg robot_name)/sonar_front</remapping>
+        </ros>
+        <output_type>sensor_msgs/Range</output_type>
+        <radiation_type>ultrasound</radiation_type>
+        <frame_name>sonar_front_link</frame_name>
+      </plugin>
+    </sensor>
+  </gazebo>
+  <!-- Sonar sensor -->
+  <gazebo reference="sonar_right_link">
+    <sensor name="sonar_right" type="ray">
+      <always_on>true</always_on>
+      <visualize>true</visualize>
+      <update_rate>60</update_rate>
+      <ray>
+        <scan>
+          <horizontal>
+            <samples>3</samples>
+            <resolution>1</resolution>
+            <min_angle>-${M_PI * 1.5/180}</min_angle>
+            <max_angle>${M_PI * 1.5/180}</max_angle>
+          </horizontal>
+          <vertical>
+            <samples>3</samples>
+            <resolution>1</resolution>
+            <min_angle>-${M_PI * 1.5/180}</min_angle>
+            <max_angle>${M_PI * 1.5/180}</max_angle>
+          </vertical>
+        </scan>
+        <range>
+          <min>0.02</min>
+          <max>20</max>
+          <resolution>0.01</resolution>
+        </range>
+        <noise>
+          <type>gaussian</type>
+          <mean>0.0</mean>
+          <stddev>0.01</stddev>
+        </noise>
+      </ray>
+      <plugin name="drone_sonar_right" filename="libgazebo_ros_ray_sensor.so">
+        <ros>
+          <remapping>~/out:=$(arg robot_name)/sonar_right</remapping>
+        </ros>
+        <output_type>sensor_msgs/Range</output_type>
+        <radiation_type>ultrasound</radiation_type>
+        <frame_name>sonar_right_link</frame_name>
+      </plugin>
+    </sensor>
+  </gazebo>
+  <gazebo reference="sonar_left_link">
+    <sensor name="sonar_left" type="ray">
+      <always_on>true</always_on>
+      <visualize>true</visualize>
+      <update_rate>60</update_rate>
+      <ray>
+        <scan>
+          <horizontal>
+            <samples>3</samples>
+            <resolution>1</resolution>
+            <min_angle>-${M_PI * 1.5/180}</min_angle>
+            <max_angle>${M_PI * 1.5/180}</max_angle>
+          </horizontal>
+          <vertical>
+            <samples>3</samples>
+            <resolution>1</resolution>
+            <min_angle>-${M_PI * 1.5/180}</min_angle>
+            <max_angle>${M_PI * 1.5/180}</max_angle>
+          </vertical>
+        </scan>
+        <range>
+          <min>0.02</min>
+          <max>20</max>
+          <resolution>0.01</resolution>
+        </range>
+        <noise>
+          <type>gaussian</type>
+          <mean>0.0</mean>
+          <stddev>0.01</stddev>
+        </noise>
+      </ray>
+      <plugin name="drone_sonar_left" filename="libgazebo_ros_ray_sensor.so">
+        <ros>
+          <remapping>~/out:=$(arg robot_name)/sonar_left</remapping>
+        </ros>
+        <output_type>sensor_msgs/Range</output_type>
+        <radiation_type>ultrasound</radiation_type>
+        <frame_name>sonar_left_link</frame_name>
+      </plugin>
+    </sensor>
+  </gazebo>
+ <gazebo reference="sonar_back_link">
+    <sensor name="sonar_back" type="ray">
+      <always_on>true</always_on>
+      <visualize>true</visualize>
+      <update_rate>60</update_rate>
+      <ray>
+        <scan>
+          <horizontal>
+            <samples>3</samples>
+            <resolution>1</resolution>
+            <min_angle>-${M_PI * 1.5/180}</min_angle>
+            <max_angle>${M_PI * 1.5/180}</max_angle>
+          </horizontal>
+          <vertical>
+            <samples>3</samples>
+            <resolution>1</resolution>
+            <min_angle>-${M_PI * 1.5/180}</min_angle>
+            <max_angle>${M_PI * 1.5/180}</max_angle>
+          </vertical>
+        </scan>
+        <range>
+          <min>0.02</min>
+          <max>20</max>
+          <resolution>0.01</resolution>
+        </range>
+        <noise>
+          <type>gaussian</type>
+          <mean>0.0</mean>
+          <stddev>0.01</stddev>
+        </noise>
+      </ray>
+      <plugin name="drone_sonar_back" filename="libgazebo_ros_ray_sensor.so">
+        <ros>
+          <remapping>~/out:=$(arg robot_name)/sonar_back</remapping>
+        </ros>
+        <output_type>sensor_msgs/Range</output_type>
+        <radiation_type>ultrasound</radiation_type>
+        <frame_name>sonar_back_link</frame_name>
       </plugin>
     </sensor>

Commit message: new launch files for a1_sup and added correct sensor link for ackerman

File: pfms-ros/audibot/audibot_description/urdf/audibot.urdf.xacro (robot description, xacro)
@@ -162,5 +162,5 @@
     <parent link="base_link" />
     <child link="laser_link" />
-    <origin xyz="${body_depth -1.05} 0 0.1" rpy="0 0 0"/>
+    <origin xyz="${body_depth -1.05} 0 0.0" rpy="0 0 0"/>
   </joint>
   <link name="laser_link"/>
@@ -171,10 +171,10 @@
   </joint>
   <link name="camera_link"/>
-  <joint name="sonar_joint" type="fixed">
+  <joint name="sonar_front_joint" type="fixed">
     <parent link="base_link" />
-    <child link="sonar_link" />
-    <origin xyz="${body_depth -1.05} 0 0.2" rpy="0 0 0"/>
+    <child link="sonar_front_link" />
+    <origin xyz="${body_depth -1.05} 0 0.3" rpy="0 0 0"/>
   </joint>
-  <link name="sonar_link"/>
+  <link name="sonar_front_link"/>
   <xacro:rear_wheel name="rl" x="${-half_wheelbase}" y="${half_rear_track_width}" z="0" flip="1" />
   <xacro:rear_wheel name="rr" x="${-half_wheelbase}" y="${-half_rear_track_width}" z="0" flip="0" />
@@ -205,5 +205,5 @@
     <sensor type='ray' name='laser'>
       <pose>0 0 0 0 0 0</pose>
-      <visualize>false</visualize>
+      <visualize>true</visualize>
       <update_rate>30</update_rate>
       <always_on>true</always_on>
@@ -282,6 +282,6 @@
   </gazebo>
   <!-- Sonar sensor -->
-  <gazebo reference="sonar_link">
-    <sensor name="sonar" type="ray">
+  <gazebo reference="sonar_front_link">
+    <sensor name="front_sonar" type="ray">
       <always_on>true</always_on>
       <visualize>true</visualize>
@@ -290,14 +290,14 @@
         <scan>
           <horizontal>
-            <samples>3</samples>
+            <samples>16</samples>
             <resolution>1</resolution>
-            <min_angle>-${M_PI * 1.5/180}</min_angle>
-            <max_angle>${M_PI * 1.5/180}</max_angle>
+            <min_angle>-${M_PI * 8/180}</min_angle>
+            <max_angle>${M_PI * 8/180}</max_angle>
           </horizontal>
           <vertical>
-            <samples>3</samples>
+            <samples>1</samples>
             <resolution>1</resolution>
-            <min_angle>-${M_PI * 1.5/180}</min_angle>
-            <max_angle>${M_PI * 1.5/180}</max_angle>
+            <min_angle>-${M_PI * 0.5/180}</min_angle>
+            <max_angle>${M_PI * 0.5/180}</max_angle>
           </vertical>
         </scan>
@@ -313,5 +313,5 @@
         </noise>
       </ray>
-      <plugin name="audi_sonar" filename="libgazebo_ros_ray_sensor.so">
+      <plugin name="audi_front_sonar" filename="libgazebo_ros_ray_sensor.so">
         <ros>
           <remapping>~/out:=$(arg robot_name)/sonar</remapping>
@@ -319,5 +319,5 @@
         <output_type>sensor_msgs/Range</output_type>
         <radiation_type>ultrasound</radiation_type>
-        <frame_name>sonar_link</frame_name>
+        <frame_name>$(arg robot_name)/sonar_front_link</frame_name>
       </plugin>
     </sensor>
