Commit message: a3 terrain simulation

File: pfms-ros/husky/husky_gazebo/urdf/husky.gazebo.xacro (robot description, xacro)
@@ -101,10 +101,10 @@
   <!-- Lidar and cameras use the general Sensors plugin -->
   <!-- DISABLED: sensors-system plugin causes segfaults with scene-broadcaster -->
-  <!-- <gazebo>
+  <gazebo>
     <plugin
         filename="libignition-gazebo-sensors-system.so"
         name="ignition::gazebo::systems::Sensors">
     </plugin>
-  </gazebo> -->
+  </gazebo>
   <gazebo reference="base_scan">
     <material>Gazebo/FlatBlack</material>
@@ -150,12 +150,12 @@
             <samples>3</samples>
             <resolution>1</resolution>
-            <min_angle>-0.026</min_angle>
-            <max_angle>0.026</max_angle>
+            <min_angle>-0.245</min_angle>
+            <max_angle>0.245</max_angle>
           </horizontal>
           <vertical>
             <samples>3</samples>
             <resolution>1</resolution>
-            <min_angle>-0.026</min_angle>
-            <max_angle>0.026</max_angle>
+            <min_angle>-0.122</min_angle>
+            <max_angle>0.122</max_angle>
           </vertical>
         </scan>

File: pfms-ros/husky/husky_gazebo/urdf/husky.urdf.xacro (robot description, xacro)
@@ -123,5 +123,5 @@
     <parent link="base_link"/>
     <child link="sonar_link"/>
-    <origin xyz="0 0 0.71" rpy="0 0 0"/>
+    <origin xyz="0 0 1.00" rpy="0 0.785398 0"/>
   </joint>
   <link name="sonar_link"/>

File: pfms-ros/husky/husky_gazebo/urdf/wheel.urdf.xacro (robot description, xacro)
@@ -14,8 +14,21 @@
       <collision>
         <origin xyz="0 0 0" rpy="1.5707963267948966 0 0"/>
-        <contact_coefficients mu="0.5" kp="1+e07" kd="1"/>
         <geometry>
           <cylinder length="0.1143" radius="${wheel_radius}"/>
         </geometry>
+        <surface>
+          <friction>
+            <ode>
+              <mu>1.0</mu>
+              <mu2>1.0</mu2>
+            </ode>
+          </friction>
+          <contact>
+            <ode>
+              <kp>1e+07</kp>
+              <kd>1.0</kd>
+            </ode>
+          </contact>
+        </surface>
       </collision>
       <inertial>

Commit message: fix for a1, position of sonar

File: pfms-ros/husky/husky_gazebo/urdf/husky.gazebo.xacro (robot description, xacro)
@@ -150,13 +150,13 @@
             <samples>3</samples>
             <resolution>1</resolution>
-            <min_angle>-0.245</min_angle>
-            <max_angle>0.245</max_angle>
+            <min_angle>-0.026</min_angle>
+            <max_angle>0.026</max_angle>
           </horizontal>
-          <!--vertical>
+          <vertical>
             <samples>3</samples>
             <resolution>1</resolution>
-            <min_angle>-0.122</min_angle>
-            <max_angle>0.122</max_angle>
-          </vertical-->
+            <min_angle>-0.026</min_angle>
+            <max_angle>0.026</max_angle>
+          </vertical>
         </scan>
         <range>

File: pfms-ros/husky/husky_gazebo/urdf/husky.urdf.xacro (robot description, xacro)
@@ -123,5 +123,5 @@
     <parent link="base_link"/>
     <child link="sonar_link"/>
-    <origin xyz="0 0 1.00" rpy="0 0.785398 0"/>
+    <origin xyz="0 0 0.71" rpy="0 0 0"/>
   </joint>
   <link name="sonar_link"/>
